File: hardware/neo-v2/kicad/Expansion.kicad_sch (KiCad schematic)
At the start: 31 parts, among them J201 OLED I2C

Commit message: NEO v2 fase 4: colocación y plan de layout
- PCB generado por script (tools/update_pcb.py) desde el PCB original de
  Nabu Casa y la netlist: contorno 84 x 89 mm con franja superior para
  batería y potencia, huellas retiradas y nuevas, zonas ampliadas,
  colocación de los bloques propios y de los puntos de prueba.
- Unión de fuentes rehecha: TPS2121 de entrada única abajo (sitio de U13)
  y LM66200 como diodo ideal en la franja, unidos por el plano +5V;
  elevador a 4,59 V. Cálculos actualizados.
- Retirados TP213 y TP221 (sin sitio); valor/DNP sincronizados.
- Huellas heredadas exportadas a kicad/lib/inherited (ERC sin avisos de
  enlace de huella).
- Paridad PCB/esquemático sin incidencias; DRC sin errores nuevos.
- docs/fase4-colocacion.md, renders, CHANGES y README.

Co-Authored-By: Claude Opus 5.5 <noreply@anthropic.com>
Claude-Session: https://claude.ai/code/session_01UWwWJAyCeb1aBHbGbkDaMx
Parts:
- removed TP221: I2S_BCLK, TestPoint:TestPoint_Pad_D1.0mm, symbol Connector:TestPoint
Other:
- note added: "PUNTOS DE PRUEBA (fase 2 §4.8): pad SMD Ø1,0 mm sobre la pista o con tramo corto (fase 4). I2S: ~0,3 pF por pad y < 1 pF por tramo, despreciable incluso para MCLK de 24,576 MHz. I2S_BCLK no tiene PT: su pista corre en el haz del bus sin hueco para un pad en ninguna cara (fase 4); se mide en el pad 2 de R71 o en el pad 1 de C128 (cara B)."
- note removed: "PUNTOS DE PRUEBA (fase 2 §4.8): pad SMD Ø1,0 mm sobre la propia pista, sin derivación. I2S: ~0,3 pF por pad, despreciable incluso para MCLK de 24,576 MHz. Si en la fase 4 no cabe un pad, el acceso será el pad de la R serie de 0 Ohm existente."
