File: hardware/neo-v2/kicad/NEO_v2.kicad_sch (KiCad schematic)
At the start: 0 parts

Commit message: hardware(neo-v2): fase 3, esquemático de bloques nuevos e integración
- Hojas nuevas Alimentacion (TPS2121, TPS61022, BQ25170, MAX17048,
  DW01A + 2x FS8205A, CSD25402Q3A, interruptor) y Expansion (conector
  OLED, pull-ups I2C, puntos de prueba), generadas por script desde
  tablas pin -> neta, referencias 201-235.
- Hojas heredadas: elimina U13 y el puerto Grove, reasigna GPIO1/2/46
  y deja sin montar R83, R84, R91 y R135; limpia hilos sueltos.
- Biblioteca propia de símbolos y huellas verificada contra los planos
  del fabricante y la huella de LCSC.
- Verificación formal de netlist contra el original y contra la
  conectividad prevista; ERC sin avisos en las hojas nuevas.
- Documentación, BOM de bloques nuevos, CHANGES.md y PDF del esquemático.

Co-Authored-By: Claude Opus 5.5 <noreply@anthropic.com>
Claude-Session: https://claude.ai/code/session_01UWwWJAyCeb1aBHbGbkDaMx
Other:
- added sheet Alimentacion (Alimentacion.kicad_sch)
- added sheet Expansion (Expansion.kicad_sch)
- note added: "NEO v2 (techmiguel), diseño derivado de Home Assistant Voice Preview Edition (Nabu Casa, CERN-OHL-P v2). Hojas de Nabu Casa: Block, ESP32, XMOS, DAC, Power, LED & Connector (cambios mínimos documentados en hardware/neo-v2/docs/fase3-esquematico.md). Hojas propias de NEO v2: Alimentacion y Expansion."
Changed lines of the file:
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@@
 		)
 	)
+	(sheet
+		(at 165.1 43.18)
+		(size 38.1 15.24)
+		(exclude_from_sim no)
+		(in_bom yes)
+		(on_board yes)
+		(dnp no)
+		(fields_autoplaced yes)
+		(stroke (width 0.1524) (type solid))
+		(fill (color 0 0 0 0.0000))
+		(property "Sheetname" "Alimentacion" (at 165.1 42.48 0) (effects (font (size 1.27 1.27)) (justify left bottom)))
+		(property "Sheetfile" "Alimentacion.kicad_sch" (at 165.1 58.980000000000004 0) (effects (font (size 1.143 1.143)) (justify left top)))
+		(instances
+			(project "NEO_v2"
+				(path "/349ed1f3-025e-4f39-9714-d91e135a7151"
+					(page "8")
+				)
+			)
+		)
+	)
+	(sheet
+		(at 165.1 68.58)
+		(size 38.1 15.24)
+		(exclude_from_sim no)
+		(in_bom yes)
+		(on_board yes)
+		(dnp no)
+		(fields_autoplaced yes)
+		(stroke (width 0.1524) (type solid))
+		(fill (color 0 0 0 0.0000))
+		(property "Sheetname" "Expansion" (at 165.1 67.88 0) (effects (font (size 1.27 1.27)) (justify left bottom)))
+		(property "Sheetfile" "Expansion.kicad_sch" (at 165.1 84.38 0) (effects (font (size 1.143 1.143)) (justify left top)))
+		(instances
+			(project "NEO_v2"
+				(path "/349ed1f3-025e-4f39-9714-d91e135a7151"
+					(page "9")
+				)
+			)
+		)
+	)
+	(text "NEO v2 (techmiguel), diseño derivado de Home Assistant Voice Preview Edition (Nabu Casa, CERN-OHL-P v2).\nHojas de Nabu Casa: Block, ESP32, XMOS, DAC, Power, LED & Connector (cambios mínimos documentados en\nhardware/neo-v2/docs/fase3-esquematico.md). Hojas propias de NEO v2: Alimentacion y Expansion." (exclude_from_sim no) (at 86.36 165.1 0) (effects (font (size 1.27 1.27)) (justify left)))
 	(sheet_instances
 		(path "/"
