File: hardware/neo-v2/kicad/NEO_v2.kicad_pcb (KiCad board)
At the start: 4 copper layers, 84 x 89 mm, 500 parts, among them J1 ST-PJ-930A, J2 WY-3315, J201 OLED I2C, Q1 CJ3407, Q10 LBSS138WT1G, Q2 LBSS138WT1G, Q201 FS8205A, Q202 FS8205A, Q203 CSD25402Q3A, Q3 LBSS138WT1G, Q4 S9013W, Q6 LBSS138WT1G, SW1 SK-22H07, SW2 AN-P1S-2SP-Z, SW201 MSK-22D18G3, SW3 MK-12C02 G1.5, U1 ESP32-S3R8, U10 TPS62827DMQR, U11 ME6211C18M5G-N, U12 TPS62065DSGR, U14 SN74LVC1G17DCKR, U15 ZB25VQ128DSJG, U16 W25Q256JVEIQ, U17 SGM7222YWQ10/TR, U18 SGM2036S-3.3XXDH4G/TR, U19 LC1458CB5TR33, U2 XU316-1024-QF60B-C24​, U201 TPS2121RUXR, U202 TPS61022RWUT, U203 BQ25170DSGR, U204 MAX17048G+T10, U205 DW01A, U206 LM66200DRLR, U3 ZB25VQ32DSJG, U4 MSM261DHP006, U5 MSM261DHP006, U6 SN74LVC125APWR, U7 SN74LVC1G17DCKR, U8 TLV320AIC3204IRHBR, U9 TPA6211A1DGNR, X1 24MHz 12pF, X2 40MHz

Commit message: NEO v2 fase 5 (en curso): ERC sin errores y ruteo de potencia
- ERC: anotaciones PWR_FLAG / no conexión sobre las hojas heredadas
  (tools/erc_annotations.py); 0 errores, solo los avisos del original.
- PCB: elevador recolocado (lazo caliente mínimo), grupo de U201 ajustado,
  ranura de SW3 estrechada y prioridad de zonas de ANT2 corregida;
  la región de rehacer de U13 conserva el VBUS de F.Cu.
- Ruteo manual de potencia (tools/route_power.py): batería, PACK_P,
  nodo SW, salida del elevador, diodo ideal, protección y U201.
- Herramientas para el autorruteo con Freerouting, cosido de GND y
  exclusiones de DRC heredadas (pendientes de aplicar).

Estado intermedio: faltan las conexiones de señal (autorruteo).

Co-Authored-By: Claude Opus 5.5 <noreply@anthropic.com>
Claude-Session: https://claude.ai/code/session_01UWwWJAyCeb1aBHbGbkDaMx
Parts:
- moved R213 18.0 mm to (197.8, 18.6)
- moved R212 15.6 mm to (197.8, 20.0)
- moved R211 13.4 mm to (197.8, 21.4)
- moved C209 8.72 mm to (194.8, 27.1), turned to -90 degrees
- moved C208 8.53 mm to (192.6, 27.1), turned to -90 degrees
- moved C206 8.42 mm to (193.6, 22.2), turned to 0 degrees
- moved C207 8.34 mm to (190.4, 27.1), turned to -90 degrees
- moved R210 5.99 mm to (195.3, 24.7)
- moved R209 5.91 mm to (195.3, 23.3), turned to 180 degrees
- moved R214 4.17 mm to (200.5, 25.9), turned to 0 degrees
- moved C205 3.55 mm to (181.0, 27.9), turned to -90 degrees
- moved C210 3.11 mm to (196.7, 27.1), turned to -90 degrees
- moved C212 2.81 mm to (205.3, 25.2), turned to -90 degrees
- moved R220 0.70 mm to (203.0, 97.7)
- moved C211 0.35 mm to (203.0, 99.5), turned to 90 degrees
Routing:
- net /Alimentacion/PACK_P: track 0.00 -> 18.4 mm
- net /Alimentacion/BOOST_5V_RAW: track 0.00 -> 13.2 mm
- net +5V: track 62.9 -> 70.7 mm, vias 29 -> 33
- net /Alimentacion/PROT_MID: track 0.00 -> 6.78 mm
- net VBUS: track 7.09 -> 13.8 mm
- net /Alimentacion/CELL_P: track 0.00 -> 6.60 mm
- net /Alimentacion/BOOST_5V: track 0.00 -> 5.48 mm
- net /Alimentacion/CELL_N: track 0.00 -> 5.43 mm
- net /Alimentacion/BOOST_FB: track 0.00 -> 4.09 mm
- net GND: track 13.0 -> 16.8 mm, vias 533 -> 537
- net /Alimentacion/BOOST_SW: track 0.00 -> 2.70 mm
Other:
- outline, holes or cut-outs redrawn
