File: hardware/neo-v2/kicad/DAC.kicad_sch (KiCad schematic)
At the start: 74 parts, among them J1 ST-PJ-930A, J2 WY-3315, Q2 LBSS138WT1G, U19 LC1458CB5TR33, U8 TLV320AIC3204IRHBR, U9 TPA6211A1DGNR

Commit message: NEO v2 fase 5 (en curso): ERC sin errores y ruteo de potencia
- ERC: anotaciones PWR_FLAG / no conexión sobre las hojas heredadas
  (tools/erc_annotations.py); 0 errores, solo los avisos del original.
- PCB: elevador recolocado (lazo caliente mínimo), grupo de U201 ajustado,
  ranura de SW3 estrechada y prioridad de zonas de ANT2 corregida;
  la región de rehacer de U13 conserva el VBUS de F.Cu.
- Ruteo manual de potencia (tools/route_power.py): batería, PACK_P,
  nodo SW, salida del elevador, diodo ideal, protección y U201.
- Herramientas para el autorruteo con Freerouting, cosido de GND y
  exclusiones de DRC heredadas (pendientes de aplicar).

Estado intermedio: faltan las conexiones de señal (autorruteo).

Co-Authored-By: Claude Opus 5.5 <noreply@anthropic.com>
Claude-Session: https://claude.ai/code/session_01UWwWJAyCeb1aBHbGbkDaMx
Changed lines of the file:
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@@
 		)
 	)
+	(symbol (lib_id "power:PWR_FLAG") (at 168.91 62.23 180) (unit 1) (exclude_from_sim no) (in_bom no) (on_board yes) (dnp no)
+		(property "Reference" "#FLG909" (at 168.91 62.23 0) (effects (font (size 1.27 1.27)) (hide yes)))
+		(property "Value" "PWR_FLAG" (at 168.91 66.04 0) (effects (font (size 1.27 1.27))))
+		(property "Footprint" "" (at 168.91 62.23 0) (effects (font (size 1.27 1.27)) (hide yes)))
+		(property "Datasheet" "" (at 168.91 62.23 0) (effects (font (size 1.27 1.27)) (hide yes)))
+		(property "Description" "NEO v2 fase 5: anotación de ERC (#PWR061)" (at 168.91 62.23 0) (effects (font (size 1.27 1.27)) (hide yes)))
+		(pin "1")
+		(instances (project "NEO_v2" (path "/349ed1f3-025e-4f39-9714-d91e135a7151/61d4d449-df96-4e92-9537-f531556a04d7" (reference "#FLG909") (unit 1))))
+	)
+	(symbol (lib_id "power:PWR_FLAG") (at 156.21 162.56 0) (unit 1) (exclude_from_sim no) (in_bom no) (on_board yes) (dnp no)
+		(property "Reference" "#FLG910" (at 156.21 162.56 0) (effects (font (size 1.27 1.27)) (hide yes)))
+		(property "Value" "PWR_FLAG" (at 156.21 158.75 0) (effects (font (size 1.27 1.27))))
+		(property "Footprint" "" (at 156.21 162.56 0) (effects (font (size 1.27 1.27)) (hide yes)))
+		(property "Datasheet" "" (at 156.21 162.56 0) (effects (font (size 1.27 1.27)) (hide yes)))
+		(property "Description" "NEO v2 fase 5: anotación de ERC (#PWR026)" (at 156.21 162.56 0) (effects (font (size 1.27 1.27)) (hide yes)))
+		(pin "1")
+		(instances (project "NEO_v2" (path "/349ed1f3-025e-4f39-9714-d91e135a7151/61d4d449-df96-4e92-9537-f531556a04d7" (reference "#FLG910") (unit 1))))
+	)
 )
