File: hardware/neo-v2/kicad/ESP32S3.kicad_sch (KiCad schematic)
At the start: 69 parts, among them U1 ESP32-S3R8, U15 ZB25VQ128DSJG, U16 W25Q256JVEIQ, X2 40MHz

Commit message: hardware(neo-v2): fase 3, esquemático de bloques nuevos e integración
- Hojas nuevas Alimentacion (TPS2121, TPS61022, BQ25170, MAX17048,
  DW01A + 2x FS8205A, CSD25402Q3A, interruptor) y Expansion (conector
  OLED, pull-ups I2C, puntos de prueba), generadas por script desde
  tablas pin -> neta, referencias 201-235.
- Hojas heredadas: elimina U13 y el puerto Grove, reasigna GPIO1/2/46
  y deja sin montar R83, R84, R91 y R135; limpia hilos sueltos.
- Biblioteca propia de símbolos y huellas verificada contra los planos
  del fabricante y la huella de LCSC.
- Verificación formal de netlist contra el original y contra la
  conectividad prevista; ERC sin avisos en las hojas nuevas.
- Documentación, BOM de bloques nuevos, CHANGES.md y PDF del esquemático.

Co-Authored-By: Claude Opus 5.5 <noreply@anthropic.com>
Claude-Session: https://claude.ai/code/session_01UWwWJAyCeb1aBHbGbkDaMx
Connections:
- net GROVE_PWR renamed ESP_IO46
- net GROVE_SCL renamed ESP_IO2
- net GROVE_SDA renamed CHG_PG
Changed lines of the file:
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@@
 		)
 	)
-	(global_label "GROVE_PWR"
+	(global_label "ESP_IO46"
 		(shape output)
 		(at 220.98 90.17 90)
@@
 		)
 	)
-	(global_label "GROVE_SDA"
+	(global_label "CHG_PG"
 		(shape bidirectional)
 		(at 160.02 124.46 180)
@@
 		)
 	)
-	(global_label "GROVE_SCL"
+	(global_label "ESP_IO2"
 		(shape output)
 		(at 160.02 127 180)

Commit message: NEO v2 fase 5 (en curso): ERC sin errores y ruteo de potencia
- ERC: anotaciones PWR_FLAG / no conexión sobre las hojas heredadas
  (tools/erc_annotations.py); 0 errores, solo los avisos del original.
- PCB: elevador recolocado (lazo caliente mínimo), grupo de U201 ajustado,
  ranura de SW3 estrechada y prioridad de zonas de ANT2 corregida;
  la región de rehacer de U13 conserva el VBUS de F.Cu.
- Ruteo manual de potencia (tools/route_power.py): batería, PACK_P,
  nodo SW, salida del elevador, diodo ideal, protección y U201.
- Herramientas para el autorruteo con Freerouting, cosido de GND y
  exclusiones de DRC heredadas (pendientes de aplicar).

Estado intermedio: faltan las conexiones de señal (autorruteo).

Co-Authored-By: Claude Opus 5.5 <noreply@anthropic.com>
Claude-Session: https://claude.ai/code/session_01UWwWJAyCeb1aBHbGbkDaMx
Connections:
- no-connect marks 6 -> 7
Changed lines of the file:
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@@
 		)
 	)
+	(symbol (lib_id "power:PWR_FLAG") (at 275.59 151.13 180) (unit 1) (exclude_from_sim no) (in_bom no) (on_board yes) (dnp no)
+		(property "Reference" "#FLG908" (at 275.59 151.13 0) (effects (font (size 1.27 1.27)) (hide yes)))
+		(property "Value" "PWR_FLAG" (at 275.59 154.94 0) (effects (font (size 1.27 1.27))))
+		(property "Footprint" "" (at 275.59 151.13 0) (effects (font (size 1.27 1.27)) (hide yes)))
+		(property "Datasheet" "" (at 275.59 151.13 0) (effects (font (size 1.27 1.27)) (hide yes)))
+		(property "Description" "NEO v2 fase 5: anotación de ERC (#PWR0199)" (at 275.59 151.13 0) (effects (font (size 1.27 1.27)) (hide yes)))
+		(pin "1")
+		(instances (project "NEO_v2" (path "/349ed1f3-025e-4f39-9714-d91e135a7151/a7f78799-685f-4ce7-bb9e-2518ac1a1bda" (reference "#FLG908") (unit 1))))
+	)
+	(no_connect (at 35.56 82.55))
 )
