File: hardware/neo-v2/kicad/LED & Connector.kicad_sch (KiCad schematic)
At the start: 101 parts, among them J4 PHS-4P, Q1 CJ3407, Q5 CJ3407, Q6 LBSS138WT1G, Q7 LBSS138WT1G, SW2 AN-P1S-2SP-Z, U20 TXS0102DCUR, U7 SN74LVC1G17DCKR

Commit message: hardware(neo-v2): fase 3, esquemático de bloques nuevos e integración
- Hojas nuevas Alimentacion (TPS2121, TPS61022, BQ25170, MAX17048,
  DW01A + 2x FS8205A, CSD25402Q3A, interruptor) y Expansion (conector
  OLED, pull-ups I2C, puntos de prueba), generadas por script desde
  tablas pin -> neta, referencias 201-235.
- Hojas heredadas: elimina U13 y el puerto Grove, reasigna GPIO1/2/46
  y deja sin montar R83, R84, R91 y R135; limpia hilos sueltos.
- Biblioteca propia de símbolos y huellas verificada contra los planos
  del fabricante y la huella de LCSC.
- Verificación formal de netlist contra el original y contra la
  conectividad prevista; ERC sin avisos en las hojas nuevas.
- Documentación, BOM de bloques nuevos, CHANGES.md y PDF del esquemático.

Co-Authored-By: Claude Opus 5.5 <noreply@anthropic.com>
Claude-Session: https://claude.ai/code/session_01UWwWJAyCeb1aBHbGbkDaMx
Parts:
- removed C100, C118, C85: 100nF, Capacitor:C0402, symbol Seeed_libadl:Capacitors/302010024
- removed C32: 10nF, Capacitor:C0402, symbol Seeed_libadl:Capacitors/302010006
- removed C84: 2.2uF, Capacitor:C0603, symbol Seeed_libdb:Capacitors/302010054
- removed C98, C99: 12pF, Capacitor:C0402, symbol Seeed_libdb:Capacitors/302010049
- removed D15, D17: ESDPSA0402V05, Diode:ESD-0402, symbol Seeed_libdb:Diode/304060074
- removed D21: TPD1E10B06DPYR, Diode:ESD-0402, symbol Seeed_libdb:Diode/304050312
- removed FB11: 120R, Inductor:L0603, symbol Seeed_libadl:Ferrite Bead/303030024
- removed J4: PHS-4P, Connector:HW4-SMD-2.0, symbol Seeed_libdb:Connector/320110030
- removed Q5: CJ3407, Mosfet:SOT23, symbol Seeed_libadl:Mosfet/305030010
- removed Q7: LBSS138WT1G, Mosfet:SOT-323, symbol Seeed_libadl:Mosfet/305031542
- removed R117, R40: 470K, Resistor:R0402, symbol Seeed_libdb:Resistors/301010069
- removed R118: 0R, Resistor:R0603, symbol Seeed_libdb:Resistors/301010292
- removed R137: 100R, Resistor:R0402, symbol Seeed_libdb:Resistors/301010028
- removed R140, R141, R144, R145, R67: 4.7K, Resistor:R0402, symbol Seeed_libdb:Resistors/301010010
- removed TP34: Test Point, Misc:TP-D45MIL, symbol libdb:Misc/TP45C_SMD
- removed U20: TXS0102DCUR, Ic:VSSOP8-0.5-2.3X2X0.9MM, symbol Seeed_libdb:Ic/310050070
- R135, R83, R84, R91: now not fitted
Connections:
- net GROVE_SCL renamed ESP_IO2
- net GROVE_SDA renamed CHG_PG

Commit message: NEO v2 fase 5 (en curso): ERC sin errores y ruteo de potencia
- ERC: anotaciones PWR_FLAG / no conexión sobre las hojas heredadas
  (tools/erc_annotations.py); 0 errores, solo los avisos del original.
- PCB: elevador recolocado (lazo caliente mínimo), grupo de U201 ajustado,
  ranura de SW3 estrechada y prioridad de zonas de ANT2 corregida;
  la región de rehacer de U13 conserva el VBUS de F.Cu.
- Ruteo manual de potencia (tools/route_power.py): batería, PACK_P,
  nodo SW, salida del elevador, diodo ideal, protección y U201.
- Herramientas para el autorruteo con Freerouting, cosido de GND y
  exclusiones de DRC heredadas (pendientes de aplicar).

Estado intermedio: faltan las conexiones de señal (autorruteo).

Co-Authored-By: Claude Opus 5.5 <noreply@anthropic.com>
Claude-Session: https://claude.ai/code/session_01UWwWJAyCeb1aBHbGbkDaMx
Changed lines of the file:
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@@
 		)
 	)
+	(symbol (lib_id "power:PWR_FLAG") (at 73.66 26.67 180) (unit 1) (exclude_from_sim no) (in_bom no) (on_board yes) (dnp no)
+		(property "Reference" "#FLG912" (at 73.66 26.67 0) (effects (font (size 1.27 1.27)) (hide yes)))
+		(property "Value" "PWR_FLAG" (at 73.66 30.48 0) (effects (font (size 1.27 1.27))))
+		(property "Footprint" "" (at 73.66 26.67 0) (effects (font (size 1.27 1.27)) (hide yes)))
+		(property "Datasheet" "" (at 73.66 26.67 0) (effects (font (size 1.27 1.27)) (hide yes)))
+		(property "Description" "NEO v2 fase 5: anotación de ERC (#PWR0189)" (at 73.66 26.67 0) (effects (font (size 1.27 1.27)) (hide yes)))
+		(pin "1")
+		(instances (project "NEO_v2" (path "/349ed1f3-025e-4f39-9714-d91e135a7151/b2f39dc0-ac44-4186-8be9-d62f5b177e00" (reference "#FLG912") (unit 1))))
+	)
 )
