File: hardware/neo-v2/kicad/XMOS.kicad_sch (KiCad schematic)
At the start: 119 parts, among them Q10 LBSS138WT1G, Q3 LBSS138WT1G, Q4 S9013W, SW1 SK-22H07, U14 SN74LVC1G17DCKR, U18 SGM2036S-3.3XXDH4G/TR, U2 XU316-1024-QF60B-C24​, U3 ZB25VQ32DSJG, U4 MSM261DHP006, U5 MSM261DHP006, U6 SN74LVC125APWR, X1 24MHz 12pF

Commit message: NEO v2 fase 5 (en curso): ERC sin errores y ruteo de potencia
- ERC: anotaciones PWR_FLAG / no conexión sobre las hojas heredadas
  (tools/erc_annotations.py); 0 errores, solo los avisos del original.
- PCB: elevador recolocado (lazo caliente mínimo), grupo de U201 ajustado,
  ranura de SW3 estrechada y prioridad de zonas de ANT2 corregida;
  la región de rehacer de U13 conserva el VBUS de F.Cu.
- Ruteo manual de potencia (tools/route_power.py): batería, PACK_P,
  nodo SW, salida del elevador, diodo ideal, protección y U201.
- Herramientas para el autorruteo con Freerouting, cosido de GND y
  exclusiones de DRC heredadas (pendientes de aplicar).

Estado intermedio: faltan las conexiones de señal (autorruteo).

Co-Authored-By: Claude Opus 5.5 <noreply@anthropic.com>
Claude-Session: https://claude.ai/code/session_01UWwWJAyCeb1aBHbGbkDaMx
Changed lines of the file:
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@@
 		)
 	)
+	(symbol (lib_id "power:PWR_FLAG") (at 69.85 46.99 0) (unit 1) (exclude_from_sim no) (in_bom no) (on_board yes) (dnp no)
+		(property "Reference" "#FLG901" (at 69.85 46.99 0) (effects (font (size 1.27 1.27)) (hide yes)))
+		(property "Value" "PWR_FLAG" (at 69.85 43.18 0) (effects (font (size 1.27 1.27))))
+		(property "Footprint" "" (at 69.85 46.99 0) (effects (font (size 1.27 1.27)) (hide yes)))
+		(property "Datasheet" "" (at 69.85 46.99 0) (effects (font (size 1.27 1.27)) (hide yes)))
+		(property "Description" "NEO v2 fase 5: anotación de ERC (U2.17 VDDIOB18)" (at 69.85 46.99 0) (effects (font (size 1.27 1.27)) (hide yes)))
+		(pin "1")
+		(instances (project "NEO_v2" (path "/349ed1f3-025e-4f39-9714-d91e135a7151/643364e4-8361-4170-9de2-28483fec4f8f" (reference "#FLG901") (unit 1))))
+	)
+	(symbol (lib_id "power:PWR_FLAG") (at 69.85 62.23 0) (unit 1) (exclude_from_sim no) (in_bom no) (on_board yes) (dnp no)
+		(property "Reference" "#FLG902" (at 69.85 62.23 0) (effects (font (size 1.27 1.27)) (hide yes)))
+		(property "Value" "PWR_FLAG" (at 69.85 58.42 0) (effects (font (size 1.27 1.27))))
+		(property "Footprint" "" (at 69.85 62.23 0) (effects (font (size 1.27 1.27)) (hide yes)))
+		(property "Datasheet" "" (at 69.85 62.23 0) (effects (font (size 1.27 1.27)) (hide yes)))
+		(property "Description" "NEO v2 fase 5: anotación de ERC (U2.4 VDD)" (at 69.85 62.23 0) (effects (font (size 1.27 1.27)) (hide yes)))
+		(pin "1")
+		(instances (project "NEO_v2" (path "/349ed1f3-025e-4f39-9714-d91e135a7151/643364e4-8361-4170-9de2-28483fec4f8f" (reference "#FLG902") (unit 1))))
+	)
+	(symbol (lib_id "power:PWR_FLAG") (at 69.85 93.98 0) (unit 1) (exclude_from_sim no) (in_bom no) (on_board yes) (dnp no)
+		(property "Reference" "#FLG903" (at 69.85 93.98 0) (effects (font (size 1.27 1.27)) (hide yes)))
+		(property "Value" "PWR_FLAG" (at 69.85 90.17 0) (effects (font (size 1.27 1.27))))
+		(property "Footprint" "" (at 69.85 93.98 0) (effects (font (size 1.27 1.27)) (hide yes)))
+		(property "Datasheet" "" (at 69.85 93.98 0) (effects (font (size 1.27 1.27)) (hide yes)))
+		(property "Description" "NEO v2 fase 5: anotación de ERC (U2.22 PLL_AVDD)" (at 69.85 93.98 0) (effects (font (size 1.27 1.27)) (hide yes)))
+		(pin "1")
+		(instances (project "NEO_v2" (path "/349ed1f3-025e-4f39-9714-d91e135a7151/643364e4-8361-4170-9de2-28483fec4f8f" (reference "#FLG903") (unit 1))))
+	)
+	(symbol (lib_id "power:PWR_FLAG") (at 19.05 254.00 180) (unit 1) (exclude_from_sim no) (in_bom no) (on_board yes) (dnp no)
+		(property "Reference" "#FLG904" (at 19.05 254.00 0) (effects (font (size 1.27 1.27)) (hide yes)))
+		(property "Value" "PWR_FLAG" (at 19.05 257.81 0) (effects (font (size 1.27 1.27))))
+		(property "Footprint" "" (at 19.05 254.00 0) (effects (font (size 1.27 1.27)) (hide yes)))
+		(property "Datasheet" "" (at 19.05 254.00 0) (effects (font (size 1.27 1.27)) (hide yes)))
+		(property "Description" "NEO v2 fase 5: anotación de ERC (#PWR0138)" (at 19.05 254.00 0) (effects (font (size 1.27 1.27)) (hide yes)))
+		(pin "1")
+		(instances (project "NEO_v2" (path "/349ed1f3-025e-4f39-9714-d91e135a7151/643364e4-8361-4170-9de2-28483fec4f8f" (reference "#FLG904") (unit 1))))
+	)
+	(symbol (lib_id "power:PWR_FLAG") (at 271.78 100.33 180) (unit 1) (exclude_from_sim no) (in_bom no) (on_board yes) (dnp no)
+		(property "Reference" "#FLG905" (at 271.78 100.33 0) (effects (font (size 1.27 1.27)) (hide yes)))
+		(property "Value" "PWR_FLAG" (at 271.78 104.14 0) (effects (font (size 1.27 1.27))))
+		(property "Footprint" "" (at 271.78 100.33 0) (effects (font (size 1.27 1.27)) (hide yes)))
+		(property "Datasheet" "" (at 271.78 100.33 0) (effects (font (size 1.27 1.27)) (hide yes)))
+		(property "Description" "NEO v2 fase 5: anotación de ERC (#PWR050)" (at 271.78 100.33 0) (effects (font (size 1.27 1.27)) (hide yes)))
+		(pin "1")
+		(instances (project "NEO_v2" (path "/349ed1f3-025e-4f39-9714-d91e135a7151/643364e4-8361-4170-9de2-28483fec4f8f" (reference "#FLG905") (unit 1))))
+	)
+	(symbol (lib_id "power:PWR_FLAG") (at 281.94 100.33 180) (unit 1) (exclude_from_sim no) (in_bom no) (on_board yes) (dnp no)
+		(property "Reference" "#FLG906" (at 281.94 100.33 0) (effects (font (size 1.27 1.27)) (hide yes)))
+		(property "Value" "PWR_FLAG" (at 281.94 104.14 0) (effects (font (size 1.27 1.27))))
+		(property "Footprint" "" (at 281.94 100.33 0) (effects (font (size 1.27 1.27)) (hide yes)))
+		(property "Datasheet" "" (at 281.94 100.33 0) (effects (font (size 1.27 1.27)) (hide yes)))
+		(property "Description" "NEO v2 fase 5: anotación de ERC (#PWR0110)" (at 281.94 100.33 0) (effects (font (size 1.27 1.27)) (hide yes)))
+		(pin "1")
+		(instances (project "NEO_v2" (path "/349ed1f3-025e-4f39-9714-d91e135a7151/643364e4-8361-4170-9de2-28483fec4f8f" (reference "#FLG906") (unit 1))))
+	)
+	(symbol (lib_id "power:PWR_FLAG") (at 396.24 219.71 180) (unit 1) (exclude_from_sim no) (in_bom no) (on_board yes) (dnp no)
+		(property "Reference" "#FLG907" (at 396.24 219.71 0) (effects (font (size 1.27 1.27)) (hide yes)))
+		(property "Value" "PWR_FLAG" (at 396.24 223.52 0) (effects (font (size 1.27 1.27))))
+		(property "Footprint" "" (at 396.24 219.71 0) (effects (font (size 1.27 1.27)) (hide yes)))
+		(property "Datasheet" "" (at 396.24 219.71 0) (effects (font (size 1.27 1.27)) (hide yes)))
+		(property "Description" "NEO v2 fase 5: anotación de ERC (#PWR075)" (at 396.24 219.71 0) (effects (font (size 1.27 1.27)) (hide yes)))
+		(pin "1")
+		(instances (project "NEO_v2" (path "/349ed1f3-025e-4f39-9714-d91e135a7151/643364e4-8361-4170-9de2-28483fec4f8f" (reference "#FLG907") (unit 1))))
+	)
 )
