File: hardware/neo-lite/kicad/NEO_Lite.kicad_sch (KiCad schematic)
At the start: 47 parts, among them J1 USB-C, J2 OLED, J3 MIC INMP441, J4 ALTAVOZ 8 Ω, J5 EXPANSIÓN, Q1 MMBT3904, Q2 MMBT3904, SW1 RESET, SW2 BOOT, U1 TLV1117LV33, U2 ESP32-S3-WROOM-1-N16R8, U3 CH340C, U4 MAX98357A

Commit message: hardware(neo-lite): fase 3, PCB y colocación
PCB de 56 x 72 mm y 2 capas creado desde la netlist (tools/build_pcb.py),
con reglas de JLCPCB, clases de neta y antena del módulo en el borde.
DRC sin errores salvo lo no ruteado. La OLED pasa a GPIO2/42 y J5 se
reordena según la salida de pines del módulo.

Co-Authored-By: Claude Opus 5.5 <noreply@anthropic.com>
Claude-Session: https://claude.ai/code/session_01T89H8KVmFbTbbN7gPJgPo2
Connections:
- net GPIO10: now also J5.15 (Pin_15); no longer J5.10 (Pin_10)
- net GPIO11: now also J5.16 (Pin_16); no longer J5.11 (Pin_11)
- net GPIO12: now also J5.17 (Pin_17); no longer J5.12 (Pin_12)
- net GPIO13: now also J5.18 (Pin_18); no longer J5.13 (Pin_13)
- net GPIO15: now also J5.9 (Pin_9); no longer J5.14 (Pin_14)
- net GPIO16: now also J5.10 (Pin_10); no longer J5.15 (Pin_15)
- net GPIO17: now also J5.11 (Pin_11); no longer J5.16 (Pin_16)
- net GPIO18: now also J5.12 (Pin_12); no longer J5.17 (Pin_17)
- net GPIO38: now also J5.19 (Pin_19); no longer J5.18 (Pin_18)
- net GPIO39: now also J5.20 (Pin_20); no longer J5.19 (Pin_19)
- net GPIO4: now also J5.5 (Pin_5); no longer J5.6 (Pin_6)
- net GPIO5: now also J5.6 (Pin_6); no longer J5.7 (Pin_7)
- net GPIO6: now also J5.7 (Pin_7); no longer J5.8 (Pin_8)
- net GPIO7: now also J5.8 (Pin_8); no longer J5.9 (Pin_9)
- net I2C_SCL: now also U2.35 (IO42); no longer U2.17 (IO9)
- net I2C_SDA: now also U2.38 (IO2); no longer U2.12 (IO8)
- removed net GPIO2: J5.5 (Pin_5), U2.38 (IO2)
- removed net GPIO42: J5.20 (Pin_20), U2.35 (IO42)
- new net GPIO8: J5.13 (Pin_13), U2.12 (IO8)
- new net GPIO9: J5.14 (Pin_14), U2.17 (IO9)
Other:
- note added: "GPIO45 y GPIO46: pines de arranque, sin carga externa. GPIO35-37: ocupados por la PSRAM octal (sin conectar). GPIO19/20 (USB nativo): solo puntos de prueba TP1/TP2. OLED en GPIO2/42 (lado derecho, junto a J2): GPIO46 debe ser 0 para la descarga."
- note removed: "GPIO45 y GPIO46: pines de arranque, sin carga externa. GPIO35-37: ocupados por la PSRAM octal (sin conectar). GPIO19/20 (USB nativo): solo puntos de prueba TP1/TP2. OLED en GPIO8/9: GPIO46 debe ser 0 para la descarga."
Changed lines of the file:
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@@
 	(label "MIC_WS" (at 264.16 83.82 180) (fields_autoplaced yes) (effects (font (size 1.27 1.27)) (justify right bottom)))
 	(wire (pts (xy 266.70 86.36) (xy 264.16 86.36)) (stroke (width 0) (type default)))
-	(label "GPIO2" (at 264.16 86.36 180) (fields_autoplaced yes) (effects (font (size 1.27 1.27)) (justify right bottom)))
+	(label "I2C_SDA" (at 264.16 86.36 180) (fields_autoplaced yes) (effects (font (size 1.27 1.27)) (justify right bottom)))
 	(wire (pts (xy 266.70 88.90) (xy 264.16 88.90)) (stroke (width 0) (type default)))
 	(label "MIC_SCK" (at 264.16 88.90 180) (fields_autoplaced yes) (effects (font (size 1.27 1.27)) (justify right bottom)))
@@
 	(label "GPIO7" (at 264.16 99.06 180) (fields_autoplaced yes) (effects (font (size 1.27 1.27)) (justify right bottom)))
 	(wire (pts (xy 266.70 101.60) (xy 264.16 101.60)) (stroke (width 0) (type default)))
-	(label "I2C_SDA" (at 264.16 101.60 180) (fields_autoplaced yes) (effects (font (size 1.27 1.27)) (justify right bottom)))
+	(label "GPIO8" (at 264.16 101.60 180) (fields_autoplaced yes) (effects (font (size 1.27 1.27)) (justify right bottom)))
 	(wire (pts (xy 266.70 104.14) (xy 264.16 104.14)) (stroke (width 0) (type default)))
-	(label "I2C_SCL" (at 264.16 104.14 180) (fields_autoplaced yes) (effects (font (size 1.27 1.27)) (justify right bottom)))
+	(label "GPIO9" (at 264.16 104.14 180) (fields_autoplaced yes) (effects (font (size 1.27 1.27)) (justify right bottom)))
 	(wire (pts (xy 266.70 106.68) (xy 264.16 106.68)) (stroke (width 0) (type default)))
 	(label "GPIO10" (at 264.16 106.68 180) (fields_autoplaced yes) (effects (font (size 1.27 1.27)) (justify right bottom)))
@@
 	(label "SPK_DIN" (at 299.72 109.22 0) (fields_autoplaced yes) (effects (font (size 1.27 1.27)) (justify left bottom)))
 	(wire (pts (xy 297.18 111.76) (xy 299.72 111.76)) (stroke (width 0) (type default)))
-	(label "GPIO42" (at 299.72 111.76 0) (fields_autoplaced yes) (effects (font (size 1.27 1.27)) (justify left bottom)))
+	(label "I2C_SCL" (at 299.72 111.76 0) (fields_autoplaced yes) (effects (font (size 1.27 1.27)) (justify left bottom)))
 	(no_connect (at 297.18 114.30))
 	(no_connect (at 297.18 116.84))
@@
 		)
 	)
-	(text "GPIO45 y GPIO46: pines de arranque, sin carga externa.\nGPIO35-37: ocupados por la PSRAM octal (sin conectar).\nGPIO19/20 (USB nativo): solo puntos de prueba TP1/TP2.\nOLED en GPIO8/9: GPIO46 debe ser 0 para la descarga." (exclude_from_sim no) (at 229.87 190.50 0) (effects (font (size 1.27 1.27)) (justify left top)))
+	(text "GPIO45 y GPIO46: pines de arranque, sin carga externa.\nGPIO35-37: ocupados por la PSRAM octal (sin conectar).\nGPIO19/20 (USB nativo): solo puntos de prueba TP1/TP2.\nOLED en GPIO2/42 (lado derecho, junto a J2): GPIO46 debe ser 0 para la descarga." (exclude_from_sim no) (at 229.87 190.50 0) (effects (font (size 1.27 1.27)) (justify left top)))
 	(text "AMPLIFICADOR I2S MAX98357A (+5V)" (exclude_from_sim no) (at 229.87 207.01 0) (effects (font (size 2.0 2.0)) (justify left top)))
 	(wire (pts (xy 259.08 236.22) (xy 256.54 236.22)) (stroke (width 0) (type default)))
@@
 		(property "Footprint" "Connector_PinHeader_2.54mm:PinHeader_1x04_P2.54mm_Vertical" (at 383.54 58.42 0) (effects (font (size 1.27 1.27)) (hide yes)))
 		(property "Datasheet" "~" (at 383.54 58.42 0) (effects (font (size 1.27 1.27)) (hide yes)))
-		(property "Description" "OLED SSD1306 0,96\" I2C (0x3C): GND, VCC, SCL, SDA" (at 383.54 58.42 0) (effects (font (size 1.27 1.27)) (hide yes)))
+		(property "Description" "OLED SSD1306 0,96\" I2C (0x3C): GND, VCC, SCL (GPIO42), SDA (GPIO2)" (at 383.54 58.42 0) (effects (font (size 1.27 1.27)) (hide yes)))
 		(pin "1")
 		(pin "2")
@@
 	)
 	(wire (pts (xy 378.46 149.86) (xy 375.92 149.86)) (stroke (width 0) (type default)))
-	(label "GPIO2" (at 375.92 149.86 180) (fields_autoplaced yes) (effects (font (size 1.27 1.27)) (justify right bottom)))
+	(label "GPIO4" (at 375.92 149.86 180) (fields_autoplaced yes) (effects (font (size 1.27 1.27)) (justify right bottom)))
 	(wire (pts (xy 378.46 152.40) (xy 375.92 152.40)) (stroke (width 0) (type default)))
-	(label "GPIO5" (at 375.92 152.40 180) (fields_autoplaced yes) (effects (font (size 1.27 1.27)) (justify right bottom)))
+	(label "GPIO6" (at 375.92 152.40 180) (fields_autoplaced yes) (effects (font (size 1.27 1.27)) (justify right bottom)))
 	(wire (pts (xy 378.46 154.94) (xy 375.92 154.94)) (stroke (width 0) (type default)))
-	(label "GPIO7" (at 375.92 154.94 180) (fields_autoplaced yes) (effects (font (size 1.27 1.27)) (justify right bottom)))
+	(label "GPIO15" (at 375.92 154.94 180) (fields_autoplaced yes) (effects (font (size 1.27 1.27)) (justify right bottom)))
 	(wire (pts (xy 378.46 157.48) (xy 375.92 157.48)) (stroke (width 0) (type default)))
-	(label "GPIO11" (at 375.92 157.48 180) (fields_autoplaced yes) (effects (font (size 1.27 1.27)) (justify right bottom)))
+	(label "GPIO17" (at 375.92 157.48 180) (fields_autoplaced yes) (effects (font (size 1.27 1.27)) (justify right bottom)))
 	(wire (pts (xy 378.46 160.02) (xy 375.92 160.02)) (stroke (width 0) (type default)))
-	(label "GPIO13" (at 375.92 160.02 180) (fields_autoplaced yes) (effects (font (size 1.27 1.27)) (justify right bottom)))
+	(label "GPIO8" (at 375.92 160.02 180) (fields_autoplaced yes) (effects (font (size 1.27 1.27)) (justify right bottom)))
 	(wire (pts (xy 378.46 162.56) (xy 375.92 162.56)) (stroke (width 0) (type default)))
-	(label "GPIO16" (at 375.92 162.56 180) (fields_autoplaced yes) (effects (font (size 1.27 1.27)) (justify right bottom)))
+	(label "GPIO10" (at 375.92 162.56 180) (fields_autoplaced yes) (effects (font (size 1.27 1.27)) (justify right bottom)))
 	(wire (pts (xy 378.46 165.10) (xy 375.92 165.10)) (stroke (width 0) (type default)))
-	(label "GPIO18" (at 375.92 165.10 180) (fields_autoplaced yes) (effects (font (size 1.27 1.27)) (justify right bottom)))
+	(label "GPIO12" (at 375.92 165.10 180) (fields_autoplaced yes) (effects (font (size 1.27 1.27)) (justify right bottom)))
 	(wire (pts (xy 378.46 167.64) (xy 375.92 167.64)) (stroke (width 0) (type default)))
-	(label "GPIO39" (at 375.92 167.64 180) (fields_autoplaced yes) (effects (font (size 1.27 1.27)) (justify right bottom)))
+	(label "GPIO38" (at 375.92 167.64 180) (fields_autoplaced yes) (effects (font (size 1.27 1.27)) (justify right bottom)))
 	(wire (pts (xy 391.16 144.78) (xy 393.70 144.78)) (stroke (width 0) (type default)))
 	(symbol
@@
 	)
 	(wire (pts (xy 391.16 149.86) (xy 393.70 149.86)) (stroke (width 0) (type default)))
-	(label "GPIO4" (at 393.70 149.86 0) (fields_autoplaced yes) (effects (font (size 1.27 1.27)) (justify left bottom)))
+	(label "GPIO5" (at 393.70 149.86 0) (fields_autoplaced yes) (effects (font (size 1.27 1.27)) (justify left bottom)))
 	(wire (pts (xy 391.16 152.40) (xy 393.70 152.40)) (stroke (width 0) (type default)))
-	(label "GPIO6" (at 393.70 152.40 0) (fields_autoplaced yes) (effects (font (size 1.27 1.27)) (justify left bottom)))
+	(label "GPIO7" (at 393.70 152.40 0) (fields_autoplaced yes) (effects (font (size 1.27 1.27)) (justify left bottom)))
 	(wire (pts (xy 391.16 154.94) (xy 393.70 154.94)) (stroke (width 0) (type default)))
-	(label "GPIO10" (at 393.70 154.94 0) (fields_autoplaced yes) (effects (font (size 1.27 1.27)) (justify left bottom)))
+	(label "GPIO16" (at 393.70 154.94 0) (fields_autoplaced yes) (effects (font (size 1.27 1.27)) (justify left bottom)))
 	(wire (pts (xy 391.16 157.48) (xy 393.70 157.48)) (stroke (width 0) (type default)))
-	(label "GPIO12" (at 393.70 157.48 0) (fields_autoplaced yes) (effects (font (size 1.27 1.27)) (justify left bottom)))
+	(label "GPIO18" (at 393.70 157.48 0) (fields_autoplaced yes) (effects (font (size 1.27 1.27)) (justify left bottom)))
 	(wire (pts (xy 391.16 160.02) (xy 393.70 160.02)) (stroke (width 0) (type default)))
-	(label "GPIO15" (at 393.70 160.02 0) (fields_autoplaced yes) (effects (font (size 1.27 1.27)) (justify left bottom)))
+	(label "GPIO9" (at 393.70 160.02 0) (fields_autoplaced yes) (effects (font (size 1.27 1.27)) (justify left bottom)))
 	(wire (pts (xy 391.16 162.56) (xy 393.70 162.56)) (stroke (width 0) (type default)))
-	(label "GPIO17" (at 393.70 162.56 0) (fields_autoplaced yes) (effects (font (size 1.27 1.27)) (justify left bottom)))
+	(label "GPIO11" (at 393.70 162.56 0) (fields_autoplaced yes) (effects (font (size 1.27 1.27)) (justify left bottom)))
 	(wire (pts (xy 391.16 165.10) (xy 393.70 165.10)) (stroke (width 0) (type default)))
-	(label "GPIO38" (at 393.70 165.10 0) (fields_autoplaced yes) (effects (font (size 1.27 1.27)) (justify left bottom)))
+	(label "GPIO13" (at 393.70 165.10 0) (fields_autoplaced yes) (effects (font (size 1.27 1.27)) (justify left bottom)))
 	(wire (pts (xy 391.16 167.64) (xy 393.70 167.64)) (stroke (width 0) (type default)))
-	(label "GPIO42" (at 393.70 167.64 0) (fields_autoplaced yes) (effects (font (size 1.27 1.27)) (justify left bottom)))
+	(label "GPIO39" (at 393.70 167.64 0) (fields_autoplaced yes) (effects (font (size 1.27 1.27)) (justify left bottom)))
 	(symbol
 		(lib_id "Connector_Generic:Conn_02x10_Odd_Even")

Commit message: hardware(neo-lite): revisión B compacta, WROOM-1U y USB nativo
Módulo ESP32-S3-WROOM-1U-N16R8 (mismas capacidades, antena externa por
U.FL), USB nativo del S3 en lugar del CH340C y el autorreset, sin la tira
de expansión J5. Placa de 31 x 43 mm (antes 56 x 72), DRC sin errores
salvo lo no ruteado; coste estimado de 72,33 USD por 5 placas.

Co-Authored-By: Claude Opus 5.5 <noreply@anthropic.com>
Claude-Session: https://claude.ai/code/session_01T89H8KVmFbTbbN7gPJgPo2
Parts:
- removed C8: 100nF, Capacitor_SMD:C_0402_1005Metric, symbol Device:C
- removed H3, H4: M3, MountingHole:MountingHole_3.2mm_M3, symbol Mechanical:MountingHole
- removed J5: EXPANSIÓN, Connector_PinHeader_2.54mm:PinHeader_2x10_P2.54mm_Vertical, symbol Connector_Generic:Conn_02x10_Odd_Even
- removed Q1, Q2: MMBT3904, Package_TO_SOT_SMD:SOT-23, symbol Transistor_BJT:MMBT3904
- removed TP4: +3V3, TestPoint:TestPoint_Pad_D1.0mm, symbol Connector:TestPoint
- removed TP5: GND, TestPoint:TestPoint_Pad_D1.0mm, symbol Connector:TestPoint
- removed TP6: U0TXD, TestPoint:TestPoint_Pad_D1.0mm, symbol Connector:TestPoint
- removed TP7: U0RXD, TestPoint:TestPoint_Pad_D1.0mm, symbol Connector:TestPoint
- removed TP8: GPIO48, TestPoint:TestPoint_Pad_D1.0mm, symbol Connector:TestPoint
- removed U3: CH340C, Package_SO:SOIC-16_3.9x9.9mm_P1.27mm, symbol NEO_Lite:CH340C_3V3
- H1, H2: value M3 -> M2; footprint MountingHole:MountingHole_3.2mm_M3 -> MountingHole:MountingHole_2.2mm_M2
- R4, R5: value 10k -> 22; LCSC C25744 -> C25092
- TP1: value USB_NAT_DP -> +5V
- TP2: value USB_NAT_DN -> +3V3
- TP3: value +5V -> GND
- U2: value ESP32-S3-WROOM-1-N16R8 -> ESP32-S3-WROOM-1U-N16R8; footprint RF_Module:ESP32-S3-WROOM-1 -> RF_Module:ESP32-S3-WROOM-1U; LCSC C2913202 -> C3013946; MPN ESP32-S3-WROOM-1-N16R8 -> ESP32-S3-WROOM-1U-N16R8
Connections:
- net DTR is gone; now on net USB_DP: R4.1
- net RTS is gone; now on net USB_DN: R5.1
- net +3V3: now also TP2.1
- net +5V: now also TP1.1; no longer TP3.1
- net GND: now also TP3.1
- net GPIO10: no longer names the net of U2.18 (IO10)
- net GPIO11: no longer names the net of U2.19 (IO11)
- net GPIO12: no longer names the net of U2.20 (IO12)
- net GPIO13: no longer names the net of U2.21 (IO13)
- net GPIO15: no longer names the net of U2.8 (IO15)
- net GPIO16: no longer names the net of U2.9 (IO16)
- net GPIO17: no longer names the net of U2.10 (IO17)
- net GPIO18: no longer names the net of U2.11 (IO18)
- net GPIO38: no longer names the net of U2.31 (IO38)
- net GPIO39: no longer names the net of U2.32 (IO39)
- net GPIO4: no longer names the net of U2.4 (IO4)
- net GPIO48: no longer names the net of U2.25 (IO48)
- net GPIO5: no longer names the net of U2.5 (IO5)
- net GPIO6: no longer names the net of U2.6 (IO6)
- net GPIO7: no longer names the net of U2.7 (IO7)
- net GPIO8: no longer names the net of U2.12 (IO8)
- net GPIO9: no longer names the net of U2.17 (IO9)
- net Q1_B renamed ESP_DP
- net ESP_DP: now also U2.14 (USB_D+)
- net Q2_B renamed ESP_DN
- net ESP_DN: now also U2.13 (USB_D-)
- net U0RXD: no longer names the net of U2.36 (RXD0)
- net U0TXD: no longer names the net of U2.37 (TXD0)
- removed net USB_NAT_DN: TP2.1, U2.13 (USB_D-)
- removed net USB_NAT_DP: TP1.1, U2.14 (USB_D+)
- no-connect marks 18 -> 30
Other:
- note added: "D+/D- del USB-C (protegidas por D1) a GPIO20/GPIO19 del módulo. Descarga y consola por el USB-Serial-JTAG integrado: sin puente USB-UART ni autorreset. Firmware: ARDUINO_USB_CDC_ON_BOOT=1. Si el firmware cuelga el USB, BOOT + RESET fuerzan la descarga."
- note added: "ESP32-S3-WROOM-1U-N16R8 (ANTENA EXTERNA U.FL)"
- note added: "GPIO45 y GPIO46: pines de arranque, sin carga externa. GPIO35-37: ocupados por la PSRAM octal (sin conectar). GPIO19/20: USB nativo (D-/D+), con R5/R4 de 22 Ω. OLED en GPIO2/42 (lado derecho, junto a J2): GPIO46 debe ser 0 para la descarga."
- note added: "J2-J4: tiras macho de 2,54 mm, cable dupont. J3: L/R del INMP441 a GND (pin 6) -> canal izquierdo (ONLY_LEFT). Antena: externa de 2,4 GHz con conector U.FL/IPEX (MHF I), al conector del módulo U2."
- note added: "USB NATIVO (USB-SERIAL-JTAG DEL ESP32-S3)"
- note removed: "Circuito de autorreset de Espressif (DevKitC): DTR RTS -> EN GPIO0 1 1 -> 1 1 0 0 -> 1 1 1 0 -> 0 1 0 1 -> 1 0 TXD de U3 -> RXD0 del ESP32 (U0RXD); RXD de U3 <- TXD0 (U0TXD)."
- note removed: "ESP32-S3-WROOM-1-N16R8"
- note removed: "GPIO45 y GPIO46: pines de arranque, sin carga externa. GPIO35-37: ocupados por la PSRAM octal (sin conectar). GPIO19/20 (USB nativo): solo puntos de prueba TP1/TP2. OLED en GPIO2/42 (lado derecho, junto a J2): GPIO46 debe ser 0 para la descarga."
- note removed: "J2-J4: tiras macho de 2,54 mm, cable dupont. J3: L/R del INMP441 a GND (pin 6) -> canal izquierdo (ONLY_LEFT). J5: sin montar. GPIO48 en TP8 (sin hueco en J5)."
- note removed: "PUENTE USB-UART (CH340C A 3,3 V) Y AUTORRESET"

Commit message: hardware(neo-lite): WROOM-1 con la antena fuera del borde en lugar del 1U
El usuario descarta la antena externa del WROOM-1U. Se vuelve al
ESP32-S3-WROOM-1-N16R8 con antena integrada, colocado con la antena
sobresaliendo del borde superior (posición recomendada por Espressif).
La placa sigue en 31 x 43 mm, DRC sin errores salvo lo no ruteado;
coste estimado de 73,14 USD por 5 placas.

Co-Authored-By: Claude Opus 5.5 <noreply@anthropic.com>
Claude-Session: https://claude.ai/code/session_01T89H8KVmFbTbbN7gPJgPo2
Parts:
- U2: value ESP32-S3-WROOM-1U-N16R8 -> ESP32-S3-WROOM-1-N16R8; footprint RF_Module:ESP32-S3-WROOM-1U -> RF_Module:ESP32-S3-WROOM-1; LCSC C3013946 -> C2913202; MPN ESP32-S3-WROOM-1U-N16R8 -> ESP32-S3-WROOM-1-N16R8
Other:
- note added: "ESP32-S3-WROOM-1-N16R8 (ANTENA PCB FUERA DEL BORDE)"
- note added: "J2-J4: tiras macho de 2,54 mm, cable dupont. J3: L/R del INMP441 a GND (pin 6) -> canal izquierdo (ONLY_LEFT). Antena: la del módulo U2, que sobresale del borde superior de la placa (guía de Espressif)."
- note removed: "ESP32-S3-WROOM-1U-N16R8 (ANTENA EXTERNA U.FL)"
- note removed: "J2-J4: tiras macho de 2,54 mm, cable dupont. J3: L/R del INMP441 a GND (pin 6) -> canal izquierdo (ONLY_LEFT). Antena: externa de 2,4 GHz con conector U.FL/IPEX (MHF I), al conector del módulo U2."
Changed lines of the file:
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@@
 	)
 	(text "D+/D- del USB-C (protegidas por D1) a GPIO20/GPIO19 del módulo.\nDescarga y consola por el USB-Serial-JTAG integrado: sin puente USB-UART ni autorreset.\nFirmware: ARDUINO_USB_CDC_ON_BOOT=1. Si el firmware cuelga el USB, BOOT + RESET fuerzan la descarga." (exclude_from_sim no) (at 20.32 229.87 0) (effects (font (size 1.27 1.27)) (justify left top)))
-	(text "ESP32-S3-WROOM-1U-N16R8 (ANTENA EXTERNA U.FL)" (exclude_from_sim no) (at 229.87 21.59 0) (effects (font (size 2.0 2.0)) (justify left top)))
+	(text "ESP32-S3-WROOM-1-N16R8 (ANTENA PCB FUERA DEL BORDE)" (exclude_from_sim no) (at 229.87 21.59 0) (effects (font (size 2.0 2.0)) (justify left top)))
 	(wire (pts (xy 266.70 76.20) (xy 264.16 76.20)) (stroke (width 0) (type default)))
 	(label "EN" (at 264.16 76.20 180) (fields_autoplaced yes) (effects (font (size 1.27 1.27)) (justify right bottom)))
@@
 		(dnp no)
 		(property "Reference" "U2" (at 269.24 72.39 0) (effects (font (size 1.27 1.27)) (justify left)))
-		(property "Value" "ESP32-S3-WROOM-1U-N16R8" (at 294.64 72.39 0) (effects (font (size 1.27 1.27)) (justify left)))
-		(property "Footprint" "RF_Module:ESP32-S3-WROOM-1U" (at 281.94 99.06 0) (effects (font (size 1.27 1.27)) (hide yes)))
+		(property "Value" "ESP32-S3-WROOM-1-N16R8" (at 294.64 72.39 0) (effects (font (size 1.27 1.27)) (justify left)))
+		(property "Footprint" "RF_Module:ESP32-S3-WROOM-1" (at 281.94 99.06 0) (effects (font (size 1.27 1.27)) (hide yes)))
 		(property "Datasheet" "https://www.espressif.com/sites/default/files/documentation/esp32-s3-wroom-1_wroom-1u_datasheet_en.pdf" (at 281.94 99.06 0) (effects (font (size 1.27 1.27)) (hide yes)))
-		(property "Description" "Módulo Wi-Fi/BLE ESP32-S3, flash 16 MB, PSRAM octal 8 MB, conector U.FL para antena externa" (at 281.94 99.06 0) (effects (font (size 1.27 1.27)) (hide yes)))
-		(property "MPN" "ESP32-S3-WROOM-1U-N16R8" (at 281.94 99.06 0) (effects (font (size 1.27 1.27)) (hide yes)))
-		(property "LCSC" "C3013946" (at 281.94 99.06 0) (effects (font (size 1.27 1.27)) (hide yes)))
+		(property "Description" "Módulo Wi-Fi/BLE ESP32-S3, flash 16 MB, PSRAM octal 8 MB, antena PCB integrada" (at 281.94 99.06 0) (effects (font (size 1.27 1.27)) (hide yes)))
+		(property "MPN" "ESP32-S3-WROOM-1-N16R8" (at 281.94 99.06 0) (effects (font (size 1.27 1.27)) (hide yes)))
+		(property "LCSC" "C2913202" (at 281.94 99.06 0) (effects (font (size 1.27 1.27)) (hide yes)))
 		(pin "3")
 		(pin "27")
@@
 		)
 	)
-	(text "J2-J4: tiras macho de 2,54 mm, cable dupont.\nJ3: L/R del INMP441 a GND (pin 6) -> canal izquierdo (ONLY_LEFT).\nAntena: externa de 2,4 GHz con conector U.FL/IPEX (MHF I), al conector del módulo U2." (exclude_from_sim no) (at 364.49 124.46 0) (effects (font (size 1.27 1.27)) (justify left top)))
+	(text "J2-J4: tiras macho de 2,54 mm, cable dupont.\nJ3: L/R del INMP441 a GND (pin 6) -> canal izquierdo (ONLY_LEFT).\nAntena: la del módulo U2, que sobresale del borde superior de la placa (guía de Espressif)." (exclude_from_sim no) (at 364.49 124.46 0) (effects (font (size 1.27 1.27)) (justify left top)))
 	(sheet_instances
 		(path "/"
