File: hardware/neo-lite/kicad/NEO_Lite.kicad_sch (KiCad schematic)
At the start: 35 parts, among them J1 USB-C, J2 OLED, J3 MIC INMP441, J4 ALTAVOZ 8 Ω, SW1 RESET, SW2 BOOT, U1 TLV1117LV33, U2 ESP32-S3-WROOM-1-N16R8, U4 MAX98357A

Commit message: hardware(neo-lite): fase 6, revisión del PCB y revisión C lista para fabricar
Revisión exhaustiva del PCB en busca de errores de concepto y de ruteo que el
DRC no detecta, con todas las correcciones aplicadas:

- Enchufado en caliente: el LC cable-cerámicos podía llevar +5V a 7-8,5 V
  (máximo absoluto de U1 y U4: 6 V). C1 pasa a tántalo AVX TPS de 47 µF/16 V
  con ESR de 0,35 Ω (C444805); tools/hotplug_sim.py lo cuantifica.
- USB-C 0,35 mm hacia dentro del borde: ahora sobresale 0,25 mm.
- Par USB sin vías y en la cara superior, con D1 en flujo continuo y R4/R5
  en el recorrido (tools/preroute.py, pistas bloqueadas).
- Desacoplo junto a los pines (C7, C9, C10) y RC de EN junto al pin EN.
- U1 girado 180° con zona de +3V3 en la lengüeta (26 mm² + lengüeta).
- Sin pistas superiores bajo el módulo; islas del plano cosidas.
- Serigrafía con trazo de 0,15 mm.

tools/review_pcb.py codifica las comprobaciones (24/24 OK) y route_all.py
solo acepta ruteos que las pasan. DRC con paridad: 0 errores, 0 pendientes.
Documentado en docs/fase6-revision.md; fases 1, 2, 4 y 5 actualizadas.

Co-Authored-By: Claude Opus 5.5 <noreply@anthropic.com>
Claude-Session: https://claude.ai/code/session_01T89H8KVmFbTbbN7gPJgPo2
Parts:
- C1: value 10uF -> 47uF 16V; footprint Capacitor_SMD:C_0805_2012Metric -> Capacitor_Tantalum_SMD:CP_EIA-6032-28_Kemet-C; symbol Device:C -> Device:C_Polarized; LCSC C15850 -> C444805; MPN (none) -> TPSC476K016R0350
Other:
- note added: "VBUS: entrada del conector (antes de F1). +5V: después de F1; alimenta U1 y el amplificador U4. R1/R2 de 5,1 kΩ: sin ellas un cargador USB-C no entrega 5 V. C1 (tántalo, ESR 0,35 Ω) amortigua la resonancia cable-cerámicos al enchufar: sin él el pico puede pasar de los 6 V máximos de U1 y U4. U1 TLV1117LV33 (no AMS1117): ver docs/fase1-componentes.md §2.3."
- note removed: "VBUS: entrada del conector (antes de F1). +5V: después de F1; alimenta U1 y el amplificador U4. R1/R2 de 5,1 kΩ: sin ellas un cargador USB-C no entrega 5 V. U1 TLV1117LV33 (no AMS1117): ver docs/fase1-componentes.md §2.3."
Changed lines of the file:
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@@
 	(title_block
 		(title "NEO Lite — ESP32-S3, micrófono, amplificador I2S y OLED")
-		(rev "A")
+		(rev "C")
 		(company "NEO — techmiguel")
 		(comment 1 "Generado por tools/gen_schematic.py: no editar a mano")
@@
 	)
 	(symbol
-		(lib_id "Device:C")
+		(lib_id "Device:C_Polarized")
 		(at 152.40 63.50 0)
 		(unit 1)
@@
 		(dnp no)
 		(property "Reference" "C1" (at 154.94 62.23 0) (effects (font (size 1.27 1.27)) (justify left)))
-		(property "Value" "10uF" (at 154.94 64.77 0) (effects (font (size 1.27 1.27)) (justify left)))
-		(property "Footprint" "Capacitor_SMD:C_0805_2012Metric" (at 152.40 63.50 0) (effects (font (size 1.27 1.27)) (hide yes)))
+		(property "Value" "47uF 16V" (at 154.94 64.77 0) (effects (font (size 1.27 1.27)) (justify left)))
+		(property "Footprint" "Capacitor_Tantalum_SMD:CP_EIA-6032-28_Kemet-C" (at 152.40 63.50 0) (effects (font (size 1.27 1.27)) (hide yes)))
 		(property "Datasheet" "~" (at 152.40 63.50 0) (effects (font (size 1.27 1.27)) (hide yes)))
-		(property "Description" "Bulk de +5V junto a la entrada" (at 152.40 63.50 0) (effects (font (size 1.27 1.27)) (hide yes)))
-		(property "LCSC" "C15850" (at 152.40 63.50 0) (effects (font (size 1.27 1.27)) (hide yes)))
+		(property "Description" "Tántalo 47 µF 16 V, ESR 0,35 Ω (AVX TPS): bulk de +5V y amortiguación del enchufado en caliente (docs/fase6-revision.md)" (at 152.40 63.50 0) (effects (font (size 1.27 1.27)) (hide yes)))
+		(property "MPN" "TPSC476K016R0350" (at 152.40 63.50 0) (effects (font (size 1.27 1.27)) (hide yes)))
+		(property "LCSC" "C444805" (at 152.40 63.50 0) (effects (font (size 1.27 1.27)) (hide yes)))
 		(pin "1")
 		(pin "2")
@@
 		)
 	)
-	(text "VBUS: entrada del conector (antes de F1).\n+5V: después de F1; alimenta U1 y el amplificador U4.\nR1/R2 de 5,1 kΩ: sin ellas un cargador USB-C no entrega 5 V.\nU1 TLV1117LV33 (no AMS1117): ver docs/fase1-componentes.md §2.3." (exclude_from_sim no) (at 119.38 95.25 0) (effects (font (size 1.27 1.27)) (justify left top)))
+	(text "VBUS: entrada del conector (antes de F1).\n+5V: después de F1; alimenta U1 y el amplificador U4.\nR1/R2 de 5,1 kΩ: sin ellas un cargador USB-C no entrega 5 V.\nC1 (tántalo, ESR 0,35 Ω) amortigua la resonancia cable-cerámicos al enchufar:\nsin él el pico puede pasar de los 6 V máximos de U1 y U4.\nU1 TLV1117LV33 (no AMS1117): ver docs/fase1-componentes.md §2.3." (exclude_from_sim no) (at 119.38 95.25 0) (effects (font (size 1.27 1.27)) (justify left top)))
 	(text "USB NATIVO (USB-SERIAL-JTAG DEL ESP32-S3)" (exclude_from_sim no) (at 20.32 147.32 0) (effects (font (size 2.0 2.0)) (justify left top)))
 	(wire (pts (xy 72.39 190.50) (xy 69.85 190.50)) (stroke (width 0) (type default)))
